File: hardware/scorbot-controller/scorbot_controller.kicad_pcb (KiCad board)
At the start: 2 copper layers, 185 x 128 mm, 113 parts, among them J1 12V in (5.5x2.1), J2 12V in (alt), J3 E-STOP (NC, in VM line), J4 DD-50 female R/A (robot cable), J5 I2C expansion, J6 Spare TCA9555 I/O, Q1 AOD4185 (rev. polarity), U1 AP63205WU, U10 Pololu #4035 DRV8874 (M1), U11 Pololu #4035 DRV8874 (M2), U12 Pololu #4035 DRV8874 (M3), U13 Pololu #4035 DRV8874 (M4), U14 Pololu #4035 DRV8874 (M5), U15 Pololu #4035 DRV8874 (M6), U2 ESP32-DevKitC-32E (38-pin), U3 74LVC14 (axes 1-3), U4 74LVC14 (axes 4-6), U5 TCA9555PWR (0x20), U6 ADS7828 (0x48)

Commit message: Swap buck, ADC and encoder buffers for plug-in modules
Replace the AP63205 buck with a Pololu D24V22F5 module, the ADS7828 with
two ADS1115 breakout modules, drop the 74LVC14 encoder buffers (4.7k
pull-ups to 3.3V straight to the ESP32) and the reverse-polarity FET.
TCA9555 stays as the only SMD IC. Module pin orders are placeholders.
Parts:
- removed C10, C12, C13, C6: 100nF, Capacitor_SMD:C_0805_2012Metric
- removed C11: 2.2uF, Capacitor_SMD:C_0805_2012Metric
- removed C4, C5: 10uF 50V, Capacitor_SMD:C_1206_3216Metric
- removed C7, C8: 22uF 10V, Capacitor_SMD:C_1206_3216Metric
- removed D2: BZT52C12 (Vgs clamp), Diode_SMD:D_SOD-123
- removed L1: 6.8uH 3A, Inductor_SMD:L_Bourns_SRN6045TA
- removed Q1: AOD4185 (rev. polarity), Package_TO_SOT_SMD:TO-252-2
- removed R1: 10k, Resistor_SMD:R_0805_2012Metric
- removed R8: 100k, Resistor_SMD:R_0805_2012Metric
- removed U3: 74LVC14 (axes 1-3), Package_SO:SOIC-14_3.9x8.7mm_P1.27mm
- removed U4: 74LVC14 (axes 4-6), Package_SO:SOIC-14_3.9x8.7mm_P1.27mm
- added U7: ADS1115 module (0x49), Scorbot:ADS1115_Module_Socket, F.Cu at (137.8, 77.8)
- D1: value SMBJ18A -> SMBJ18A (unidirectional)
- R40, R41, R42, R43, R44, R45, R46, R47, R48, R49, R50, R51: value 10k -> 4.7k
- U1: value AP63205WU -> Pololu D24V22F5 (5V 2.5A); footprint Package_TO_SOT_SMD:TSOT-23-6 -> Scorbot:Pololu_D24V22F5_Socket
- U6: value ADS7828 (0x48) -> ADS1115 module (0x48); footprint Package_SO:TSSOP-16_4.4x5mm_P0.65mm -> Scorbot:ADS1115_Module_Socket
- moved C50 32.3 mm to (184.1, 89.5)
- moved R51 32.3 mm to (188.7, 89.4)
- moved C51 32.3 mm to (193.3, 89.5)
- moved C65 29.2 mm to (164.3, 144.2)
- moved R65 29.2 mm to (159.7, 144.2)
- moved R5 27.1 mm to (50.3, 70.7)
- moved R6 27.1 mm to (54.9, 70.7)
- moved R4 27.1 mm to (45.7, 70.7)
- moved C42 27.0 mm to (159.7, 82.5)
- moved R43 27.0 mm to (164.4, 82.5)
- moved D5 25.3 mm to (76.3, 93.8)
- moved D4 25.3 mm to (69.9, 93.0)
- moved C47 23.1 mm to (179.4, 86.0)
- moved R47 23.1 mm to (174.8, 86.0)
- moved R48 23.1 mm to (189.8, 86.0)
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Connections:
- F1 pad 2: VIN_F -> VIN
- R40 pad 1: +5V -> +3V3
- R41 pad 1: +5V -> +3V3
- R42 pad 1: +5V -> +3V3
- R43 pad 1: +5V -> +3V3
- R44 pad 1: +5V -> +3V3
- R45 pad 1: +5V -> +3V3
- R46 pad 1: +5V -> +3V3
- R47 pad 1: +5V -> +3V3
- R48 pad 1: +5V -> +3V3
- R49 pad 1: +5V -> +3V3
- R50 pad 1: +5V -> +3V3
- R51 pad 1: +5V -> +3V3
- U1 pad 1: +5V -> (no net)
- U1 pad 2: BUCK_EN -> VIN
- U1 pad 3: VIN -> GND
- U1 pad 4: GND -> +5V
- U2 pad 10: ENC4_B -> ENC4_P1
- U2 pad 11: ENC5_A -> ENC5_P0
- U2 pad 15: ENC5_B -> ENC5_P1
- U2 pad 21: ENC6_B -> ENC6_P1
- U2 pad 3: ENC1_A -> ENC1_P0
- U2 pad 32: ENC6_A -> ENC6_P0
- U2 pad 4: ENC1_B -> ENC1_P1
- U2 pad 5: ENC2_A -> ENC2_P0
- U2 pad 6: ENC2_B -> ENC2_P1
- U2 pad 7: ENC3_A -> ENC3_P0
- U2 pad 8: ENC3_B -> ENC3_P1
- U2 pad 9: ENC4_A -> ENC4_P0
- U6 pad 1: CS1 -> +3V3
- U6 pad 10: ADC_REF -> CS4
- U6 pad 2: CS2 -> GND
- U6 pad 3: CS3 -> SCL
- U6 pad 4: CS4 -> SDA
- U6 pad 5: CS5 -> GND
- U6 pad 6: CS6 -> (no net)
- U6 pad 7: VM_ADC -> CS1
- U6 pad 8: GND -> CS2
- U6 pad 9: GND -> CS3
