File: hardware/scorbot-controller/scorbot_controller.kicad_pcb (KiCad board)
At the start: 2 copper layers, 185 x 128 mm, 98 parts, among them J1 12V in (5.5x2.1), J2 12V in (alt), J3 E-STOP (NC, in VM line), J4 DD-50 female R/A (robot cable), J5 I2C expansion, J6 Spare TCA9555 I/O, U1 Pololu D24V22F5 (5V 2.5A), U10 Pololu #4035 DRV8874 (M1), U11 Pololu #4035 DRV8874 (M2), U12 Pololu #4035 DRV8874 (M3), U13 Pololu #4035 DRV8874 (M4), U14 Pololu #4035 DRV8874 (M5), U15 Pololu #4035 DRV8874 (M6), U2 ESP32-DevKitC-32E (38-pin), U5 TCA9555PWR (0x20), U6 ADS1115 module (0x48), U7 ADS1115 module (0x49)

Commit message: Board rev: screw terminals for fuse and E-stop, 4-pin DROK buck socket
Fuse holder replaced by a screw terminal (wire an inline fuse across it),
E-stop plug replaced by a screw terminal, buck module socket now IN+, IN-,
OUT-, OUT+ to match the DROK mini buck. Barrel jack footprint matched to
CUI PJ-102AH. ADS1115 socket follows Adafruit #1085. DevKit relabelled for
WROOM-32D or -32E (same pins).

Co-Authored-By: Claude Opus 5.5 <noreply@anthropic.com>
Claude-Session: https://claude.ai/code/session_01EVE6PZ95cMufMkAr9pDFuN
Parts:
- removed F1: 5A blade (mini), Fuse:Fuseholder_Blade_Mini_Keystone_3568
- added J7: FUSE (wire inline 5A fuse across), TerminalBlock_Phoenix:TerminalBlock_Phoenix_MKDS-1,5-2-5.08_1x02_P5.08mm_Horizontal, F.Cu at (34.1, 72.8)
- J1: value 12V in (5.5x2.1) -> 12V in (CUI PJ-102AH, 2.1 mm); footprint Connector_BarrelJack:BarrelJack_Horizontal -> Connector_BarrelJack:BarrelJack_CUI_PJ-102AH_Horizontal
- J3: footprint Connector_Phoenix_MSTB:PhoenixContact_MSTBA_2,5_2-G-5,08_1x02_P5.08mm_Horizontal -> TerminalBlock_Phoenix:TerminalBlock_Phoenix_MKDS-1,5-2-5.08_1x02_P5.08mm_Horizontal
- U1: value Pololu D24V22F5 (5V 2.5A) -> DROK mini buck, set to 5V; footprint Scorbot:Pololu_D24V22F5_Socket -> Scorbot:Buck_Module_4pin_Socket
- U2: value ESP32-DevKitC-32E (38-pin) -> ESP32-DevKitC (WROOM-32D or -32E, 38-pin)
- moved R4 37.3 mm to (78.5, 53.0)
- moved R5 37.3 mm to (83.1, 53.0)
- moved C3 11.0 mm to (50.3, 64.8)
- moved R6 11.0 mm to (45.7, 64.7)
- moved R7 11.0 mm to (55.0, 64.7)
- moved D3 11.0 mm to (59.6, 64.8)
- moved R2 8.49 mm to (68.7, 53.1)
- moved C1 8.49 mm to (52.8, 57.3)
- moved C2 8.49 mm to (63.5, 53.0)
- moved D1 8.49 mm to (46.3, 55.7)
- moved R3 8.49 mm to (73.9, 53.0)
- moved D4 6.00 mm to (75.9, 93.0)
- moved D5 6.00 mm to (82.3, 93.8)
- moved R9 6.00 mm to (71.2, 93.0)
- moved J3 5.49 mm to (34.1, 91.1)
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Connections:
- U1 pad 1: (no net) -> VIN
- U1 pad 2: VIN -> GND
