File: hardware/scorbot-controller/scorbot_controller.kicad_sch (KiCad schematic)
At the start: 113 parts, among them J1 12V in (5.5x2.1), J2 12V in (alt), J3 E-STOP (NC, in VM line), J4 DD-50 female R/A (robot cable), J5 I2C expansion, J6 Spare TCA9555 I/O, Q1 AOD4185 (rev. polarity), U1 AP63205WU, U10 Pololu #4035 DRV8874 (M1), U11 Pololu #4035 DRV8874 (M2), U12 Pololu #4035 DRV8874 (M3), U13 Pololu #4035 DRV8874 (M4), U14 Pololu #4035 DRV8874 (M5), U15 Pololu #4035 DRV8874 (M6), U2 ESP32-DevKitC-32E (38-pin), U3 74LVC14 (axes 1-3), U4 74LVC14 (axes 4-6), U5 TCA9555PWR (0x20), U6 ADS7828 (0x48)

Commit message: Swap buck, ADC and encoder buffers for plug-in modules
Replace the AP63205 buck with a Pololu D24V22F5 module, the ADS7828 with
two ADS1115 breakout modules, drop the 74LVC14 encoder buffers (4.7k
pull-ups to 3.3V straight to the ESP32) and the reverse-polarity FET.
TCA9555 stays as the only SMD IC. Module pin orders are placeholders.
Parts:
- removed C10, C12, C13, C6: 100nF, Capacitor_SMD:C_0805_2012Metric, symbol Device:C
- removed C11: 2.2uF, Capacitor_SMD:C_0805_2012Metric, symbol Device:C
- removed C4, C5: 10uF 50V, Capacitor_SMD:C_1206_3216Metric, symbol Device:C
- removed C7, C8: 22uF 10V, Capacitor_SMD:C_1206_3216Metric, symbol Device:C
- removed D2: BZT52C12 (Vgs clamp), Diode_SMD:D_SOD-123, symbol Device:D_Zener
- removed L1: 6.8uH 3A, Inductor_SMD:L_Bourns_SRN6045TA, symbol Device:L
- removed Q1: AOD4185 (rev. polarity), Package_TO_SOT_SMD:TO-252-2, symbol Device:Q_PMOS_GDS
- removed R1: 10k, Resistor_SMD:R_0805_2012Metric, symbol Device:R
- removed R8: 100k, Resistor_SMD:R_0805_2012Metric, symbol Device:R
- removed U3: 74LVC14 (axes 1-3), Package_SO:SOIC-14_3.9x8.7mm_P1.27mm, symbol 74xx:74HC14
- removed U4: 74LVC14 (axes 4-6), Package_SO:SOIC-14_3.9x8.7mm_P1.27mm, symbol 74xx:74HC14
- added U7: ADS1115 module (0x49), Scorbot:ADS1115_Module_Socket, symbol Scorbot:ADS1115_Module
- D1: value SMBJ18A -> SMBJ18A (unidirectional)
- R40, R41, R42, R43, R44, R45, R46, R47, R48, R49, R50, R51: value 10k -> 4.7k
- U1: value AP63205WU -> Pololu D24V22F5 (5V 2.5A); footprint Package_TO_SOT_SMD:TSOT-23-6 -> Scorbot:Pololu_D24V22F5_Socket; symbol Regulator_Switching:AP63205WU -> Scorbot:Pololu_D24V22F5
- U6: value ADS7828 (0x48) -> ADS1115 module (0x48); footprint Package_SO:TSSOP-16_4.4x5mm_P0.65mm -> Scorbot:ADS1115_Module_Socket; symbol Analog_ADC:ADS7828 -> Scorbot:ADS1115_Module
Connections:
- net ADC_REF is gone; now on net CS4: U6.10 (A3)
- net BUCK_EN is gone; now on net VIN: U1.2 (VIN)
- net ENC1_A is gone; now on net ENC1_P0: U2.3 (IO36)
- net ENC1_B is gone; now on net ENC1_P1: U2.4 (IO39)
- net ENC2_A is gone; now on net ENC2_P0: U2.5 (IO34)
- net ENC2_B is gone; now on net ENC2_P1: U2.6 (IO35)
- net ENC3_A is gone; now on net ENC3_P0: U2.7 (IO32)
- net ENC3_B is gone; now on net ENC3_P1: U2.8 (IO33)
- net ENC4_A is gone; now on net ENC4_P0: U2.9 (IO25)
- net ENC4_B is gone; now on net ENC4_P1: U2.10 (IO26)
- net ENC5_A is gone; now on net ENC5_P0: U2.11 (IO27)
- net ENC5_B is gone; now on net ENC5_P1: U2.15 (IO13)
- net ENC6_A is gone; now on net ENC6_P0: U2.32 (IO4)
- net ENC6_B is gone; now on net ENC6_P1: U2.21 (IO23)
- net VIN_F is gone; now on net VIN: F1.2
- net +3V3: now also R40.1, R41.1, R42.1, R43.1, R44.1, R45.1, R46.1, R47.1, R48.1, R49.1, R50.1, R51.1, U6.1 (VDD), U7.1 (VDD), U7.5 (ADDR); no longer U6.16 (VDD)
- net +5V: now also U1.4 (VOUT); no longer R40.1, R41.1, R42.1, R43.1, R44.1, R45.1, R46.1, R47.1, R48.1, R49.1, R50.1, R51.1, U1.1 (FB)
- net CS1: now also U6.7 (A0); no longer U6.1 (CH0)
- net CS2: now also U6.8 (A1); no longer U6.2 (CH1)
- net CS3: now also U6.9 (A2); no longer U6.3 (CH2)
- net CS4: no longer U6.4 (CH3)
- net CS5: now also U7.7 (A0); no longer U6.5 (CH4)
- net CS6: now also U7.8 (A1); no longer U6.6 (CH5)
- net GND: now also U1.3 (GND), U6.2 (GND), U6.5 (ADDR), U7.10 (A3), U7.2 (GND); no longer U1.4 (GND), U6.11 (COM), U6.12 (A0), U6.13 (A1), U6.8 (CH7), U6.9 (GND)
- net SCL: now also U6.3 (SCL), U7.3 (SCL); no longer U6.14 (SCL)
- net SDA: now also U6.4 (SDA), U7.4 (SDA); no longer U6.15 (SDA)
- net VIN: no longer U1.3 (IN)
- net VM_ADC: now also U7.9 (A2); no longer U6.7 (CH6)
- removed net BUCK_BST: U1.6 (BST)
- removed net BUCK_SW: U1.5 (SW)
- no-connect marks 31 -> 34
Other:
- moved on the sheet: C1, C2, C21, C22, C23, C24, C25, C26, C3, C40, C41, C42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
