File: hardware/scorbot-controller/scorbot_controller.kicad_sch (KiCad schematic)
At the start: 98 parts, among them J1 12V in (5.5x2.1), J2 12V in (alt), J3 E-STOP (NC, in VM line), J4 DD-50 female R/A (robot cable), J5 I2C expansion, J6 Spare TCA9555 I/O, U1 Pololu D24V22F5 (5V 2.5A), U10 Pololu #4035 DRV8874 (M1), U11 Pololu #4035 DRV8874 (M2), U12 Pololu #4035 DRV8874 (M3), U13 Pololu #4035 DRV8874 (M4), U14 Pololu #4035 DRV8874 (M5), U15 Pololu #4035 DRV8874 (M6), U2 ESP32-DevKitC-32E (38-pin), U5 TCA9555PWR (0x20), U6 ADS1115 module (0x48), U7 ADS1115 module (0x49)

Commit message: Update schematic notes for the module-based design
Co-Authored-By: Claude Opus 5.5 <noreply@anthropic.com>
Claude-Session: https://claude.ai/code/session_01EVE6PZ95cMufMkAr9pDFuN
Other:
- note added: "5 V: Pololu D24V22F5 plug-in buck + DEVKIT 5V FEED"
- note added: "ENCODER FRONT END: 47R VLED from 5V, 4.7k pull-ups to 3.3V, 1nF, direct to ESP32"
- note added: "I2C: TCA9555 (0x20) + 2x ADS1115 modules (0x48, 0x49)"
- note added: "NOTES 1. Pololu DRV8874 carrier pin ORDER is a placeholder (names are correct). Fix design.CARRIER_ROWS and regenerate. 2. DB50 pinout from SCORBOT-ER 4u User Manual ch. 8 (same as ER III Table D-1). Pins 37-44 unused, 22 = gripper switch (no connection in arm). 3. Plug-in module pin orders (Pololu D24V22F5, ADS1115 breakout) are placeholders: check against your modules. 4. Carrier current limit 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"
- note removed: "5 V BUCK + DEVKIT 5V FEED"
- note removed: "ENCODER FRONT END: 47R VLED, 10k pull-ups to 5V, 1nF, 74LVC14 at 3.3V"
- note removed: "I2C: TCA9555 (0x20) + ADS7828 (0x48)"
- note removed: "NOTES 1. Pololu DRV8874 carrier pin ORDER is a placeholder (names are correct). Fix design.CARRIER_ROWS and regenerate. 2. DB50 pinout from SCORBOT-ER 4u User Manual ch. 8 (same as ER III Table D-1). Pins 37-44 unused, 22 = gripper switch (no connection in arm). 3. 74HC14 symbol is used for the 74LVC14 (same pinout). Powered from +3V3; inputs are 5 V tolerant. 4. Carrier current limit with SLEEP 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"
Changed lines of the file:
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@@
     (effects (font (size 1.8 1.8) bold) (justify left))
   )
-  (text "5 V BUCK + DEVKIT 5V FEED" (at 226.41900000000004 20 0)
+  (text "5 V: Pololu D24V22F5 plug-in buck + DEVKIT 5V FEED"
+    (at 226.41900000000004 20 0)
     (effects (font (size 1.8 1.8) bold) (justify left))
   )
@@
     (effects (font (size 1.8 1.8) bold) (justify left))
   )
-  (text "I2C: TCA9555 (0x20) + ADS7828 (0x48)" (at 491.427 20 0)
+  (text "I2C: TCA9555 (0x20) + 2x ADS1115 modules (0x48, 0x49)"
+    (at 491.427 20 0)
     (effects (font (size 1.8 1.8) bold) (justify left))
   )
@@
     (effects (font (size 1.8 1.8) bold) (justify left))
   )
-  (text "ENCODER FRONT END: 47R VLED, 10k pull-ups to 5V, 1nF, 74LVC14 at 3.3V"
+  (text "ENCODER FRONT END: 47R VLED from 5V, 4.7k pull-ups to 3.3V, 1nF, direct to ESP32"
     (at 334.06800000000004 157.14 0)
     (effects (font (size 1.8 1.8) bold) (justify left))
@@
     (effects (font (size 1.8 1.8) bold) (justify left))
   )
-  (text "NOTES\n1. Pololu DRV8874 carrier pin ORDER is a placeholder (names are correct). Fix design.CARRIER_ROWS and regenerate.\n2. DB50 pinout from SCORBOT-ER 4u User Manual ch. 8 (same as ER III Table D-1). Pins 37-44 unused, 22 = gripper switch (no connection in arm).\n3. 74HC14 symbol is used for the 74LVC14 (same pinout). Powered from +3V3; inputs are 5 V tolerant.\n4. Carrier current limit with SLEEP at 3.3 V is about 2.9 A (VREF pulled to SLEEP by 10k on the carrier, CS has 2.49k). R21-R26 (DNP) lower it.\n5. ADS7828 uses its internal 2.5 V reference: CS reads 1.12 V/A, so readings clip above about 2.2 A."
+  (text "NOTES\n1. Pololu DRV8874 carrier pin ORDER is a placeholder (names are correct). Fix design.CARRIER_ROWS and regenerate.\n2. DB50 pinout from SCORBOT-ER 4u User Manual ch. 8 (same as ER III Table D-1). Pins 37-44 unused, 22 = gripper switch (no connection in arm).\n3. Plug-in module pin orders (Pololu D24V22F5, ADS1115 breakout) are placeholders: check against your modules.\n4. Carrier current limit with SLEEP at 3.3 V is about 2.9 A (VREF pulled to SLEEP by 10k on the carrier, CS has 2.49k). R21-R26 (DNP) lower it.\n5. Current sense: CS reads 1.12 V/A into ADS1115 modules (use the +/-4.096 V range). VM monitored via 47k/10k on ADS1115 #2 A2."
     (at 15 340.52 0)
     (effects (font (size 1.8 1.8) bold) (justify left))

Commit message: Board rev: screw terminals for fuse and E-stop, 4-pin DROK buck socket
Fuse holder replaced by a screw terminal (wire an inline fuse across it),
E-stop plug replaced by a screw terminal, buck module socket now IN+, IN-,
OUT-, OUT+ to match the DROK mini buck. Barrel jack footprint matched to
CUI PJ-102AH. ADS1115 socket follows Adafruit #1085. DevKit relabelled for
WROOM-32D or -32E (same pins).

Co-Authored-By: Claude Opus 5.5 <noreply@anthropic.com>
Claude-Session: https://claude.ai/code/session_01EVE6PZ95cMufMkAr9pDFuN
Parts:
- removed F1: 5A blade (mini), Fuse:Fuseholder_Blade_Mini_Keystone_3568, symbol Device:Fuse
- added J7: FUSE (wire inline 5A fuse across), TerminalBlock_Phoenix:TerminalBlock_Phoenix_MKDS-1,5-2-5.08_1x02_P5.08mm_Horizontal, symbol Connector:Screw_Terminal_01x02
- J1: value 12V in (5.5x2.1) -> 12V in (CUI PJ-102AH, 2.1 mm); footprint Connector_BarrelJack:BarrelJack_Horizontal -> Connector_BarrelJack:BarrelJack_CUI_PJ-102AH_Horizontal
- J3: footprint Connector_Phoenix_MSTB:PhoenixContact_MSTBA_2,5_2-G-5,08_1x02_P5.08mm_Horizontal -> TerminalBlock_Phoenix:TerminalBlock_Phoenix_MKDS-1,5-2-5.08_1x02_P5.08mm_Horizontal
- U1: value Pololu D24V22F5 (5V 2.5A) -> DROK mini buck, set to 5V; footprint Scorbot:Pololu_D24V22F5_Socket -> Scorbot:Buck_Module_4pin_Socket; symbol Scorbot:Pololu_D24V22F5 -> Scorbot:Buck_Module_4pin
- U2: value ESP32-DevKitC-32E (38-pin) -> ESP32-DevKitC (WROOM-32D or -32E, 38-pin)
Connections:
- net GND: now also U1.2 (IN-)
- net VIN: now also U1.1 (IN+), J7.2 (Pin_2); no longer U1.2 (VIN)
- net VIN_RAW: now also J7.1 (Pin_1)
- no-connect marks 34 -> 33
Other:
- note added: "5 V: DROK buck module in 4-pin socket (IN+ IN- OUT- OUT+) + DEVKIT 5V FEED"
- note added: "ESP32-DevKitC, WROOM-32D or -32E (plug-in, 2x 1x19 female headers)"
- note added: "NOTES 1. Pololu DRV8874 carrier pin ORDER is a placeholder (names are correct). Fix design.CARRIER_ROWS and regenerate. 2. DB50 pinout from SCORBOT-ER 4u User Manual ch. 8 (same as ER III Table D-1). Pins 37-44 unused, 22 = gripper switch (no connection in arm). 3. Buck socket follows the DROK module (EN unused). ADS1115 socket follows Adafruit #1085; other boards differ. 4. Carrier current limit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"
- note removed: "5 V: Pololu D24V22F5 plug-in buck + DEVKIT 5V FEED"
- note removed: "ESP32-DevKitC-32E (plug-in, 2x 1x19 female headers)"
- note removed: "NOTES 1. Pololu DRV8874 carrier pin ORDER is a placeholder (names are correct). Fix design.CARRIER_ROWS and regenerate. 2. DB50 pinout from SCORBOT-ER 4u User Manual ch. 8 (same as ER III Table D-1). Pins 37-44 unused, 22 = gripper switch (no connection in arm). 3. Plug-in module pin orders (Pololu D24V22F5, ADS1115 breakout) are placeholders: check against your modules. 4. Carrier current limit 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"
- moved on the sheet: C1, C2, C3, C9, D1, D3, D4, D5, D6, D7, J1, J2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
