File: hardware/scorbot-controller/scorbot_controller.kicad_sch (KiCad schematic)
At the start: 98 parts, among them J1 12V in (CUI PJ-102AH, 2.1 mm), J2 12V in (alt), J3 E-STOP (NC, in VM line), J4 DD-50 female R/A (robot cable), J5 I2C expansion, J6 Spare TCA9555 I/O, J7 FUSE (wire inline 5A fuse acr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, U1 DROK mini buck, set to 5V, U10 Pololu #4035 DRV8874 (M1), U11 Pololu #4035 DRV8874 (M2), U12 Pololu #4035 DRV8874 (M3), U13 Pololu #4035 DRV8874 (M4), U14 Pololu #4035 DRV8874 (M5), U15 Pololu #4035 DRV8874 (M6), U2 ESP32-DevKitC (WROOM-32D or -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, U5 TCA9555PWR (0x20), U6 ADS1115 module (0x48), U7 ADS1115 module (0x49)

Commit message: Board: screw-terminal power input beside the barrel jack, optional on-board blade fuse holder
- J2 is now a plain 5.08 mm screw terminal (alternative to barrel jack J1)
- F1 Keystone 3568 mini blade holder in parallel with the J7 fuse terminal; fit one
- Net classes for Power/Motor/Supply; gen_route.py autoroutes with Freerouting
Parts:
- added F1: 5A mini blade (Keystone 3568 holder), Fuse:Fuseholder_Blade_Mini_Keystone_3568, symbol Device:Fuse
- J2: value 12V in (alt) -> 12V in (screw terminal, +/-); footprint Connector_Phoenix_MSTB:PhoenixContact_MSTBA_2,5_2-G-5,08_1x02_P5.08mm_Horizontal -> TerminalBlock_Phoenix:TerminalBlock_Phoenix_MKDS-1,5-2-5.08_1x02_P5.08mm_Horizontal
- J7: value FUSE (wire inline 5A fuse across) -> FUSE alt: wire inline 5A fuse (fit F1 OR J7)
Connections:
- net VIN: now also F1.2
- net VIN_RAW: now also F1.1
Other:
- moved on the sheet: C1, C2, C3, C9, D1, D3, D4, D5, D6, D7, J3, J5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

Commit message: v0.3: verified carrier pinout, on-board ADS1115s, wider power traces, SMD or THT TVS
- DRV8874 carrier socket from Pololu's labeled top view (2x7, 0.5in rows),
  VM/VIN orientation marks on the silkscreen
- ADS1115IDGSR x2 placed by JLC (0x48/0x49 by ADDR strap) replace the plug-in
  modules; 100nF decoupling each
- 1 oz copper: VIN/VM 2.5 mm with 1.6/0.8 mm vias, motor 1.2 mm with 1.2/0.6 mm vias
- D1 SMBJ18A (SMB) or D8 1.5KE18A (DO-201AD THT), hand-fitted, out of the JLC BOM
- JLC BOM grouped by LCSC part; README: how to check part numbers and orientation
Parts:
- added C10, C11: 100nF, Capacitor_SMD:C_0805_2012Metric, symbol Device:C
- added D8: 1.5KE18A THT (fit D1 OR D8), Diode_THT:D_DO-201AD_P15.24mm_Horizontal, symbol Device:D_TVS
- D1: value SMBJ18A (unidirectional) -> SMBJ18A (fit D1 OR D8)
- U6: value ADS1115 module (0x48) -> ADS1115IDGSR (0x48); footprint Scorbot:ADS1115_Module_Socket -> Package_SO:TSSOP-10_3x3mm_P0.5mm; symbol Scorbot:ADS1115_Module -> Analog_ADC:ADS1115IDGS
- U7: value ADS1115 module (0x49) -> ADS1115IDGSR (0x49); footprint Scorbot:ADS1115_Module_Socket -> Package_SO:TSSOP-10_3x3mm_P0.5mm; symbol Scorbot:ADS1115_Module -> Analog_ADC:ADS1115IDGS
Connections:
- net +3V3: now also U6.8 (VDD), U7.8 (VDD), C10.1, C11.1; no longer U6.1 (VDD), U7.5 (ADDR)
- net CS1: now also U10.14 (CS), U6.4 (AIN0); no longer U10.13 (CS), U6.7 (A0)
- net CS2: now also U11.14 (CS), U6.5 (AIN1); no longer U11.13 (CS), U6.8 (A1)
- net CS3: now also U12.14 (CS), U6.6 (AIN2); no longer U12.13 (CS), U6.9 (A2)
- net CS4: now also U13.14 (CS), U6.7 (AIN3); no longer U13.13 (CS), U6.10 (A3)
- net CS5: now also U14.14 (CS), U7.4 (AIN0); no longer U14.13 (CS), U7.7 (A0)
- net CS6: now also U15.14 (CS), U7.5 (AIN1); no longer U15.13 (CS), U7.8 (A1)
- net GND: now also U10.2 (GND), U10.5 (PMODE), U10.9 (GND), U11.2 (GND), U11.5 (PMODE), U11.9 (GND), U12.2 (GND), U12.5 (PMODE), U12.9 (GND), U13.2 (GND), U13.5 (PMODE), U13.9 (GND), U14.2 (GND), U14.5 (PMODE), U14.9 (GND), U15.2 (GND), U15.5 (PMODE), U15.9 (GND), U6.1 (ADDR), U6.3 (GND), U7.3 (GND), U7.7 (AIN3), C10.2, C11.2, D8.2 (A2); no longer U10.3 (GND), U10.6 (GND), U10.7 (PMODE), U11.3 (GND), U11.6 (GND), U11.7 (PMODE), U12.3 (GND), U12.6 (GND), U12.7 (PMODE), U13.3 (GND), U13.6 (GND), U13.7 (PMODE), U14.3 (GND), U14.6 (GND), U14.7 (PMODE), U15.3 (GND), U15.6 (GND), U15.7 (PMODE), U6.2 (GND), U6.5 (ADDR), U7.10 (A3), U7.2 (GND)
- net MOT1_A: now also U10.10 (OUT1); no longer U10.4 (OUT1)
- net MOT1_B: now also U10.11 (OUT2); no longer U10.5 (OUT2)
- net MOT2_A: now also U11.10 (OUT1); no longer U11.4 (OUT1)
- net MOT2_B: now also U11.11 (OUT2); no longer U11.5 (OUT2)
- net MOT3_A: now also U12.10 (OUT1); no longer U12.4 (OUT1)
- net MOT3_B: now also U12.11 (OUT2); no longer U12.5 (OUT2)
- net MOT4_A: now also U13.10 (OUT1); no longer U13.4 (OUT1)
- net MOT4_B: now also U13.11 (OUT2); no longer U13.5 (OUT2)
- net MOT5_A: now also U14.10 (OUT1); no longer U14.4 (OUT1)
- net MOT5_B: now also U14.11 (OUT2); no longer U14.5 (OUT2)
- net MOT6_A: now also U15.10 (OUT1); no longer U15.4 (OUT1)
- net MOT6_B: now also U15.11 (OUT2); no longer U15.5 (OUT2)
- net NFAULT: now also U10.13 (FAULT), U11.13 (FAULT), U12.13 (FAULT), U13.13 (FAULT), U14.13 (FAULT), U15.13 (FAULT); no longer U10.12 (FAULT), U11.12 (FAULT), U12.12 (FAULT), U13.12 (FAULT), U14.12 (FAULT), U15.12 (FAULT)
- net NSLEEP: now also U10.6 (SLEEP), U11.6 (SLEEP), U12.6 (SLEEP), U13.6 (SLEEP), U14.6 (SLEEP), U15.6 (SLEEP); no longer U10.11 (SLEEP), U11.11 (SLEEP), U12.11 (SLEEP), U13.11 (SLEEP), U14.11 (SLEEP), U15.11 (SLEEP)
- net PH1: now also U10.4 (PH); no longer U10.10 (PH)
- net PH2: now also U11.4 (PH); no longer U11.10 (PH)
- net PH3: now also U12.4 (PH); no longer U12.10 (PH)
- net PH4: now also U13.4 (PH); no longer U13.10 (PH)
- net PH5: now also U14.4 (PH); no longer U14.10 (PH)
- net PH6: now also U15.4 (PH); no longer U15.10 (PH)
- net PWM1: now also U10.3 (EN); no longer U10.9 (EN)
- net PWM2: now also U11.3 (EN); no longer U11.9 (EN)
- net PWM3: now also U12.3 (EN); no longer U12.9 (EN)
- net PWM4: now also U13.3 (EN); no longer U13.9 (EN)
- net PWM5: now also U14.3 (EN); no longer U14.9 (EN)
- net PWM6: now also U15.3 (EN); no longer U15.9 (EN)
- net SCL: now also U6.10 (SCL), U7.10 (SCL); no longer U6.3 (SCL), U7.3 (SCL)
- net SDA: now also U6.9 (SDA), U7.9 (SDA); no longer U6.4 (SDA), U7.4 (SDA)
- net VIN: now also D8.1 (A1)
- net VM: now also U10.8 (VIN), U11.8 (VIN), U12.8 (VIN), U13.8 (VIN), U14.8 (VIN), U15.8 (VIN); no longer U10.1 (VIN), U11.1 (VIN), U12.1 (VIN), U13.1 (VIN), U14.1 (VIN), U15.1 (VIN)
- net VM_ADC: now also U7.6 (AIN2); no longer U7.9 (A2)
- net VREF1: now also U10.7 (VREF); no longer U10.14 (VREF)
- net VREF2: now also U11.7 (VREF); no longer U11.14 (VREF)
- net VREF3: now also U12.7 (VREF); no longer U12.14 (VREF)
- net VREF4: now also U13.7 (VREF); no longer U13.14 (VREF)
- net VREF5: now also U14.7 (VREF); no longer U14.14 (VREF)
- net VREF6: now also U15.7 (VREF); no longer U15.14 (VREF)
Other:
- moved on the sheet: C1, C2, C21, C22, C23, C24, C25, C26, C3, C40, C41, C42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
