File: hardware/drv8874-carrier/drv8874_carrier_b.kicad_pcb (KiCad board)
At the start: 2 copper layers, 15.2 x 17.8 mm, 11 parts, among them J1 1x7 0.1in pins (hand-soldered), J2 1x7 0.1in pins (hand-soldered), U1 DRV8874PWPR

Commit message: DRV8874 carrier: Basic parts only besides the DRV8874, add C4
- C1, C2: 10 uF 25 V 0805 (C15850) instead of 50 V 1206 (C13585), much
  cheaper.
- C5: 22 nF 0402 (C1532, Basic) instead of 0603 (C77571, Extended).
- R3: 2.4 k (C22940, Basic) instead of 2.49 k. CS reads 1.08 V/A and the
  driver limit is about 3.1 A.
- C4: second 100 nF on VM, by the VM header pin, as on Pololu's board.
- A no-tracks rule area keeps signals from under U1 on B.Cu, so the
  thermal pad's bottom pour is unbroken. Version B now gets all 15
  thermal vias.
- R3's GND pad gets its own via. GND is no longer widened (it is poured).

Firmware: the driver choice is now a menuconfig choice between this
carrier (default, 1.08 V/A), Pololu #4035 (1.12 V/A) and #4036
(2.49 V/A). Host tests pass for all three.
Parts:
- added C4: 100nF 50V, C_0603_1608Metric, F.Cu at (103.4, 103.0)
- C1, C2: value 10uF 50V -> 10uF 25V; footprint C_1206_3216Metric -> C_0805_2012Metric
- C5: footprint C_0603_1608Metric -> C_0402_1005Metric
- R3: value 2.49k 1% -> 2.4k 1%
- moved C1 0.70 mm to (106.8, 103.0)
- moved C2 0.45 mm to (110.2, 103.0)
Routing:
- net FAULT: track 28.3 -> 9.58 mm, vias 3 -> 1
- net GND: track 54.3 -> 46.7 mm, vias 11 -> 12
- net IMODE: track 10.2 -> 8.55 mm
- net SLEEP: track 7.25 -> 8.80 mm, vias 1 -> 0
- net VM: track 38.0 -> 39.0 mm
- net VREF: track 12.2 -> 11.4 mm, vias 1 -> 2
